Commit message: Tested three robot convoy repeat on a simulated mesh of UTIAS

File: src/hunter_sim/hunter2_base/urdf/hunter2_base_gazebo_lidar.xacro (robot description, xacro)
@@ -153,5 +153,6 @@
     <axis
       xyz="0 0 -1" />
-    <limit effort="10" velocity="100" />
+    <limit effort="300" velocity="100" />
+    <dynamics friction="0.0" damping="0.0"/>
   </joint>
   <link
@@ -262,5 +263,6 @@
     <axis
       xyz="0 0 -1" />
-    <limit effort="10" velocity="100" />
+    <limit effort="300" velocity="100" />
+    <dynamics friction="0.0" damping="0.0"/>
   </joint>
   <link
@@ -315,5 +317,6 @@
     <axis
       xyz="0 0 -1" />
-    <limit effort="10" velocity="100" />
+    <limit effort="300" velocity="100" />
+    <dynamics friction="1.0" damping="1.0"/>
   </joint>
   <link
@@ -368,5 +371,6 @@
     <axis
       xyz="0 0 -1" />
-    <limit effort="10" velocity="100" />
+    <limit effort="300" velocity="100" />
+    <dynamics friction="1.0" damping="1.0"/>
   </joint>
   <link

File: src/hunter_sim/hunter2_base/urdf/hunter2_base_gazebo_lidar_2.xacro (robot description, xacro)
@@ -153,5 +153,6 @@
     <axis
       xyz="0 0 -1" />
-    <limit effort="10" velocity="100" />
+    <limit effort="300" velocity="100" />
+    <dynamics friction="0.0" damping="0.0"/>
   </joint>
   <link
@@ -262,5 +263,6 @@
     <axis
       xyz="0 0 -1" />
-    <limit effort="10" velocity="100" />
+    <limit effort="300" velocity="100" />
+    <dynamics friction="0.0" damping="0.0"/>
   </joint>
   <link
@@ -315,5 +317,6 @@
     <axis
       xyz="0 0 -1" />
-    <limit effort="10" velocity="100" />
+    <limit effort="300" velocity="100" />
+    <dynamics friction="1.0" damping="1.0"/>
   </joint>
   <link
@@ -368,5 +371,6 @@
     <axis
       xyz="0 0 -1" />
-    <limit effort="10" velocity="100" />
+    <limit effort="300" velocity="100" />
+    <dynamics friction="1.0" damping="1.0"/>
   </joint>
   <link
