Commit message: WIP harmonic updates to use non-deprecated modes

File: src/hunter_sim/hunter2_base/urdf/hunter2_base_gazebo.xacro (robot description, xacro)
@@ -3,501 +3,284 @@
      Commit Version: 1.6.0-1-g15f4949  Build Version: 1.6.7594.29634
      For more information, please see http://wiki.ros.org/sw_urdf_exporter -->
-<robot name="hunter2" xmlns:xacro="http://www.ros.org/wiki/xacro">
-<xacro:include filename="$(find hunter2_gazebo)/xacro/hunter2.gazebo"/>
-  <link
-    name="base_link">
-    <inertial>
-      <origin
-        xyz="0.0266989327622036 0.000409203500587652 -0.135901124750884"
-        rpy="0 0 0" />
-      <mass
-        value="10" />
-      <inertia
-        ixx="0.0332370959804736"
-        ixy="-1.013150489971E-06"
-        ixz="-0.00188859201421112"
-        iyy="0.111072002332437"
-        iyz="-5.13308150598312E-07"
-        izz="0.12660862809283" />
-    </inertial>
-    <visual>
-      <origin
-        xyz="0 0 0"
-        rpy="0 0 0" />
-      <geometry>
-        <mesh
-          filename="file://$(find hunter2_base)/meshes/base_link.STL" />
-      </geometry>
-      <material
-        name="">
-        <color
-          rgba="0.792156862745098 0.819607843137255 0.933333333333333 1" />
-      </material>
-    </visual>
-    <collision>
-      <origin
-        xyz="0 0 0"
-        rpy="0 0 0" />
-      <geometry>
-        <mesh
-          filename="file://$(find hunter2_base)/meshes/base_link.STL" />
-      </geometry>
-    </collision>
-  </link>
-  <link
-    name="front_steer_left_link">
-    <inertial>
-      <origin
-        xyz="-0.012614 1.8116E-05 0.0023132"
-        rpy="0 0 0" />
-      <mass
-        value="0.5" />
-      <inertia
-        ixx="0.0222"
-        ixy="0.0"
-        ixz="0.0"
-        iyy="0.0222"
-        iyz="0.0"
-        izz="0.0378075" />
-    </inertial>
-    <visual>
-      <origin
-        xyz="0 0 0"
-        rpy="0 0 0" />
-      <geometry>
-        <box size="0.001 0.001 0.001"/>
-      </geometry>
-      <material
-        name="">
-        <color
-          rgba="0.79216 0.81961 0.93333 1" />
-      </material>
-    </visual>
-    <collision>
-      <origin
-        xyz="0 0 0"
-        rpy="0 0 0" />
-      <geometry>
-        <box size="0.001 0.001 0.001"/>
-      </geometry>
-    </collision>
-  </link>
-  <joint
-    name="front_steer_left_joint"
-    type="continuous">
-    <origin
-      xyz="0.37142 0.29199 -0.1955"
-      rpy="1.5708 0 0" />
-    <parent
-      link="base_link" />
-    <child
-      link="front_steer_left_link" />
-    <axis
-      xyz="0 1 0" />
-    <limit
-      lower="-0.69"
-      upper="0.69"
-      effort="10"
-      velocity="0.69" />
-  </joint>
-  <link
-    name="front_left_wheel_link">
-    <inertial>
-      <origin
-        xyz="-6.5774E-06 2.0242E-05 -0.0096386"
-        rpy="0 0 0" />
-      <mass
-        value="1" />
-      <inertia
-        ixx="0.063724"
-        ixy="0"
-        ixz="0"
-        iyy="0.063724"
-        iyz="0"
-        izz="0.11072" />
-    </inertial>
-    <visual>
-      <origin
-        xyz="0 0 0"
-        rpy="0 0 0" />
-      <geometry>
-        <mesh
-          filename="file://$(find hunter2_base)/meshes/front_left_wheel_link.STL" />
-      </geometry>
-      <material
-        name="">
-        <color
-          rgba="0.79216 0.81961 0.93333 1" />
-      </material>
-    </visual>
-    <collision>
-      <origin
-        xyz="0 0 0"
-        rpy="0 0 0" />
-      <geometry>
-        <cylinder radius="0.165" length="0.14"/>
-      </geometry>
-    </collision>
-  </link>
-  <joint
-    name="front_left_wheel_joint"
-    type="continuous">
-    <origin
-      xyz="0 0 0"
-      rpy="0 0 0" />
-    <parent
-      link="front_steer_left_link" />
-    <child
-      link="front_left_wheel_link" />
-    <axis
-      xyz="0 0 -1" />
-    <limit effort="10" velocity="100" />
-  </joint>
-  <link
-    name="front_steer_right_link">
-    <inertial>
-      <origin
-        xyz="-8.9374E-08 1.0997E-07 0.0095958"
-        rpy="0 0 0" />
-      <mass
-        value="0.5" />
-      <inertia
-        ixx="0.0222"
-        ixy="0.0"
-        ixz="0.0"
-        iyy="0.0222"
-        iyz="0.0"
-        izz="0.0378075" />
-    </inertial>
-    <visual>
-      <origin
-        xyz="0 0 0"
-        rpy="0 0 0" />
-      <geometry>
-        <box size="0.001 0.001 0.001"/>
-      </geometry>
-      <material
-        name="">
-        <color
-          rgba="0.79216 0.81961 0.93333 1" />
-      </material>
-    </visual>
-    <collision>
-      <origin
-        xyz="0 0 0"
-        rpy="0 0 0" />
-      <geometry>
-        <box size="0.001 0.001 0.001"/>
-      </geometry>
-    </collision>
-  </link>
-  <joint
-    name="front_steer_right_joint"
-    type="continuous">
-    <origin
-      xyz="0.37142 -0.29201 -0.1955"
-      rpy="1.5708 0 0" />
-    <parent
-      link="base_link" />
-    <child
-      link="front_steer_right_link" />
-    <axis
-      xyz="0 1 0" />
-    <limit
-      lower="-0.69"
-      upper="0.69"
-      effort="10"
-      velocity="0.69" />
-  </joint>
-  <link
-    name="front_right_wheel_link">
-    <inertial>
-      <origin
-        xyz="-9.1148E-08 1.1284E-07 0.0095049"
-        rpy="0 0 0" />
-      <mass
-        value="1" />
-      <inertia
-        ixx="0.063626"
-        ixy="0"
-        ixz="0"
-        iyy="0.063626"
-        iyz="0"
-        izz="0.11054" />
-    </inertial>
-    <visual>
-      <origin
-        xyz="0 0 0"
-        rpy="0 3.14 0" />
-      <geometry>
-        <mesh
-          filename="file://$(find hunter2_base)/meshes/front_left_wheel_link.STL" />
-      </geometry>
-      <material
-        name="">
-        <color
-          rgba="0.79216 0.81961 0.93333 1" />
-      </material>
-    </visual>
-    <collision>
-      <origin
-        xyz="0 0 0"
-        rpy="0 0 0" />
-      <geometry>
-        <cylinder radius="0.165" length="0.14"/>
-      </geometry>
-    </collision>
-  </link>
-  <joint
-    name="front_right_wheel_joint"
-    type="continuous">
-    <origin
-      xyz="0 0 0"
-      rpy="0 0 0" />
-    <parent
-      link="front_steer_right_link" />
-    <child
-      link="front_right_wheel_link" />
-    <axis
-      xyz="0 0 -1" />
-    <limit effort="10" velocity="100" />
-  </joint>
-  <link
-    name="rear_left_link">
-    <inertial>
-      <origin
-        xyz="-8.826E-05 6.4342E-05 -0.0096491"
-        rpy="0 0 0" />
-      <mass
-        value="1" />
-      <inertia
-        ixx="0.063699"
-        ixy="0"
-        ixz="0"
-        iyy="0.063699"
-        iyz="0"
-        izz="0.11067" />
-    </inertial>
-    <visual>
-      <origin
-        xyz="0 0 0"
-        rpy="0 0 0" />
-      <geometry>
-        <mesh
-          filename="file://$(find hunter2_base)/meshes/left_rear_link.STL" />
-      </geometry>
-      <material
-        name="">
-        <color
-          rgba="0.79216 0.81961 0.93333 1" />
-      </material>
-    </visual>
-    <collision>
-      <origin
-        xyz="0 0 0"
-        rpy="0 0 0" />
-      <geometry>
-        <cylinder radius="0.165" length="0.14"/>
-      </geometry>
-    </collision>
-  </link>
-  <joint
-    name="rear_left_joint"
-    type="continuous">
-    <origin
-      xyz="-0.28 0.29249 -0.19558"
-      rpy="1.5708 0 0" />
-    <parent
-      link="base_link" />
-    <child
-      link="rear_left_link" />
-    <axis
-      xyz="0 0 -1" />
-    <limit effort="10" velocity="100" />
-  </joint>
-  <link
-    name="rear_right_link">
-    <inertial>
-      <origin
-        xyz="8.6344E-05 7.4488E-05 0.0097824"
-        rpy="0 0 0" />
-      <mass
-        value="1" />
-      <inertia
-        ixx="0.06373"
-        ixy="0"
-        ixz="0"
-        iyy="0.06373"
-        iyz="0"
-        izz="0.11073" />
-    </inertial>
-    <visual>
-      <origin
-        xyz="0 0 0"
-        rpy="0 0 0" />
-      <geometry>
-        <mesh
-          filename="file://$(find hunter2_base)/meshes/right_rear_link.STL" />
-      </geometry>
-      <material
-        name="">
-        <color
-          rgba="0.79216 0.81961 0.93333 1" />
-      </material>
-    </visual>
-    <collision>
-      <origin
-        xyz="0 0 0"
-        rpy="0 0 0" />
-      <geometry>
-         <cylinder radius="0.165" length="0.14"/>
-      </geometry>
-    </collision>
-  </link>
-  <joint
-    name="rear_right_joint"
-    type="continuous">
-    <origin
-      xyz="-0.28018 -0.29251 -0.19558"
-      rpy="1.5708 0.0026575 0" />
-    <parent
-      link="base_link" />
-    <child
-      link="rear_right_link" />
-    <axis
-      xyz="0 0 -1" />
-    <limit effort="10" velocity="100" />
-  </joint>
-  <link
-    name="front_steer_link">
-    <inertial>
-      <origin
-        xyz="0.049836 8.1046E-15 0.017912"
-        rpy="0 0 0" />
-      <mass
-        value="0.049179" />
-      <inertia
-        ixx="1.6846E-07"
-        ixy="7.6396E-23"
-        ixz="-1.0974E-08"
-        iyy="7.549E-07"
-        iyz="-1.8957E-22"
-        izz="7.334E-07" />
-    </inertial>
-    <visual>
-      <origin
-        xyz="0 0 0"
-        rpy="0 0 0" />
-      <geometry>
-      <cylinder length="0.001" radius="0.005"/>
-      </geometry>
-      <material
-        name="">
-        <color
-          rgba="0.79216 0.81961 0.93333 1" />
-      </material>
-    </visual>
-    <collision>
-      <origin
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
File: src/hunter_sim/hunter2_base/urdf/hunter2_base_gazebo_lidar.xacro (robot description, xacro)
@@ -4,6 +4,6 @@
      For more information, please see http://wiki.ros.org/sw_urdf_exporter -->
 <robot name="hunter2" xmlns:xacro="http://www.ros.org/wiki/xacro">
-<xacro:include filename="$(find hunter2_gazebo)/xacro/lidar.xacro" />
-<xacro:include filename="$(find hunter2_gazebo)/xacro/hunter2.gazebo"/>
+<xacro:include filename="package://hunter2_gazebo/xacro/lidar.xacro" />
+<xacro:include filename="package://hunter2_gazebo/xacro/hunter2.gazebo"/>
   <link
     name="base_link">
@@ -28,5 +28,5 @@
       <geometry>
         <mesh
-          filename="file://$(find hunter2_base)/meshes/base_link.STL" />
+          filename="package://hunter2_base/meshes/base_link.STL" />
       </geometry>
       <material
@@ -42,5 +42,5 @@
       <geometry>
         <mesh
-          filename="file://$(find hunter2_base)/meshes/base_link.STL" />
+          filename="package://hunter2_base/meshes/base_link.STL" />
       </geometry>
     </collision>
@@ -124,5 +124,5 @@
       <geometry>
         <mesh
-          filename="file://$(find hunter2_base)/meshes/front_left_wheel_link.STL" />
+          filename="package://hunter2_base/meshes/front_left_wheel_link.STL" />
       </geometry>
       <material
@@ -234,5 +234,5 @@
       <geometry>
         <mesh
-          filename="file://$(find hunter2_base)/meshes/front_left_wheel_link.STL" />
+          filename="package://hunter2_base/meshes/front_left_wheel_link.STL" />
       </geometry>
       <material
@@ -288,5 +288,5 @@
       <geometry>
         <mesh
-          filename="file://$(find hunter2_base)/meshes/left_rear_link.STL" />
+          filename="package://hunter2_base/meshes/left_rear_link.STL" />
       </geometry>
       <material
@@ -342,5 +342,5 @@
       <geometry>
         <mesh
-          filename="file://$(find hunter2_base)/meshes/right_rear_link.STL" />
+          filename="package://hunter2_base/meshes/right_rear_link.STL" />
       </geometry>
       <material

File: src/hunter_sim/hunter2_base/urdf/hunter2_base_gazebo_lidar_2.xacro (robot description, xacro)
@@ -4,6 +4,6 @@
      For more information, please see http://wiki.ros.org/sw_urdf_exporter -->
 <robot name="hunter2" xmlns:xacro="http://www.ros.org/wiki/xacro">
-<xacro:include filename="$(find hunter2_gazebo)/xacro/lidar.xacro" />
-<xacro:include filename="$(find hunter2_gazebo)/xacro/hunter2_2.gazebo"/>
+<xacro:include filename="package://hunter2_gazebo/xacro/lidar.xacro" />
+<xacro:include filename="package://hunter2_gazebo/xacro/hunter2_2.gazebo"/>
   <link
     name="base_link">
@@ -28,5 +28,5 @@
       <geometry>
         <mesh
-          filename="file://$(find hunter2_base)/meshes/base_link.STL" />
+          filename="package://hunter2_base/meshes/base_link.STL" />
       </geometry>
       <material
@@ -42,5 +42,5 @@
       <geometry>
         <mesh
-          filename="file://$(find hunter2_base)/meshes/base_link.STL" />
+          filename="package://hunter2_base/meshes/base_link.STL" />
       </geometry>
     </collision>
@@ -124,5 +124,5 @@
       <geometry>
         <mesh
-          filename="file://$(find hunter2_base)/meshes/front_left_wheel_link.STL" />
+          filename="package://hunter2_base/meshes/front_left_wheel_link.STL" />
       </geometry>
       <material
@@ -234,5 +234,5 @@
       <geometry>
         <mesh
-          filename="file://$(find hunter2_base)/meshes/front_left_wheel_link.STL" />
+          filename="package://hunter2_base/meshes/front_left_wheel_link.STL" />
       </geometry>
       <material
@@ -288,5 +288,5 @@
       <geometry>
         <mesh
-          filename="file://$(find hunter2_base)/meshes/left_rear_link.STL" />
+          filename="package://hunter2_base/meshes/left_rear_link.STL" />
       </geometry>
       <material
@@ -342,5 +342,5 @@
       <geometry>
         <mesh
-          filename="file://$(find hunter2_base)/meshes/right_rear_link.STL" />
+          filename="package://hunter2_base/meshes/right_rear_link.STL" />
       </geometry>
       <material

File: src/hunter_sim/hunter2_base/urdf/hunter2_base_gazebo_lidar_3.xacro (robot description, xacro)
@@ -4,6 +4,6 @@
      For more information, please see http://wiki.ros.org/sw_urdf_exporter -->
 <robot name="hunter2" xmlns:xacro="http://www.ros.org/wiki/xacro">
-<xacro:include filename="$(find hunter2_gazebo)/xacro/lidar.xacro" />
-<xacro:include filename="$(find hunter2_gazebo)/xacro/hunter2_3.gazebo"/>
+<xacro:include filename="package://hunter2_gazebo/xacro/lidar.xacro" />
+<xacro:include filename="package://hunter2_gazebo/xacro/hunter2_3.gazebo"/>
   <link
     name="base_link">
@@ -28,5 +28,5 @@
       <geometry>
         <mesh
-          filename="file://$(find hunter2_base)/meshes/base_link.STL" />
+          filename="package://hunter2_base/meshes/base_link.STL" />
       </geometry>
       <material
@@ -42,5 +42,5 @@
       <geometry>
         <mesh
-          filename="file://$(find hunter2_base)/meshes/base_link.STL" />
+          filename="package://hunter2_base/meshes/base_link.STL" />
       </geometry>
     </collision>
@@ -124,5 +124,5 @@
       <geometry>
         <mesh
-          filename="file://$(find hunter2_base)/meshes/front_left_wheel_link.STL" />
+          filename="package://hunter2_base/meshes/front_left_wheel_link.STL" />
       </geometry>
       <material
@@ -234,5 +234,5 @@
       <geometry>
         <mesh
-          filename="file://$(find hunter2_base)/meshes/front_left_wheel_link.STL" />
+          filename="package://hunter2_base/meshes/front_left_wheel_link.STL" />
       </geometry>
       <material
@@ -288,5 +288,5 @@
       <geometry>
         <mesh
-          filename="file://$(find hunter2_base)/meshes/left_rear_link.STL" />
+          filename="package://hunter2_base/meshes/left_rear_link.STL" />
       </geometry>
       <material
@@ -342,5 +342,5 @@
       <geometry>
         <mesh
-          filename="file://$(find hunter2_base)/meshes/right_rear_link.STL" />
+          filename="package://hunter2_base/meshes/right_rear_link.STL" />
       </geometry>
       <material
